Commit message: +update camera

File: ros2_differential_drive_robot/install/ros2_differential_drive_robot/share/ros2_differential_drive_robot/description/camera.xacro (robot description, xacro)
@@ -4,4 +4,5 @@
         <parent link="chassis"/>
         <child link="camera_link"/>
+        <!-- <origin xyz="0.0 0.0 0.08" rpy="0.0 0.0 0.0"/> -->
         <origin xyz="0.305 0.0 0.08" rpy="0.0 0.0 0.0"/>
     </joint>
@@ -38,12 +39,12 @@
           <far>300</far>
         </clip>
-        <noise>
-          <type>gaussian</type>
+        <!-- <noise> -->
+          <!-- <type>gaussian</type> -->
           <!-- Noise is sampled independently per pixel on each frame.
                That pixel's noise value is added to each of its color
                channels, which at that point lie in the range [0,1]. -->
-          <mean>0.0</mean>
-          <stddev>0.007</stddev>
-        </noise>
+          <!-- <mean>0.0</mean> -->
+          <!-- <stddev>0.007</stddev> -->
+        <!-- </noise> -->
       </camera>
       <plugin name="camera_controller" filename="libgazebo_ros_camera.so">
