Commit message: + added new project

File: ros2_differential_obstacle_robot/install/rover/share/rover/description/robot.urdf.xacro (robot description, xacro)
@@ -1,8 +1,9 @@
 <?xml version="1.0"?>
 <robot xmlns:xacro="http://www.ros.org/wiki/xacro" name="rover">
-  <xacro:include filename="robot_core.xacro"/>
+  <xacro:include filename="rover.xacro"/>
+  <!-- <xacro:include filename="robot_core.xacro"/> -->
   <!-- <xacro:include filename="gazebo_control_skid_steering.xacro"/> -->
-  <xacro:include filename="camera.xacro" />
-  <xacro:include filename="lidar.xacro" />
-  <xacro:include filename="gazebo_control_differential_drive.xacro" />
+  <!-- <xacro:include filename="camera.xacro" /> -->
+  <!-- <xacro:include filename="lidar.xacro" /> -->
+  <!-- <xacro:include filename="gazebo_control_differential_drive.xacro" /> -->
 </robot>

File: ros2_differential_obstacle_robot/install/rover/share/rover/description/robot_core.xacro (robot description, xacro)
@@ -1,5 +1,4 @@
 <?xml version="1.0"?>
 <robot xmlns:xacro="http://www.ros.org/wiki/xacro" name="rover">
-    <xacro:include filename="inertial_macros.xacro"/>
     <material name="white">
         <color rgba="1 1 1 1"/>
@@ -17,8 +16,15 @@
         <color rgba="1 0 0 1"/>
     </material>
-    <link name="chassis">
+    <link name="base_link"></link>
+    <joint name="base_link_joint" type="fixed">
+        <origin xyz="0.0 0.0 0.1" rpy="0.0 0.0 0.0"/>
+        <parent link="base_link"/>
+        <child link="chassis_link"/>
+        <axis xyz="0.0 0.0 0.0"/>
+    </joint>
+    <link name="chassis_link">
         <visual>
             <geometry>
-                <box size=".8 0.7 0.1"/>
+                <box size="0.8 0.7 0.2"/>
             </geometry>
             <material name="orange"/>
@@ -26,46 +32,15 @@
         <collision>
             <geometry>
-                <box size=".8 0.7 0.1"/>
+                <box size="0.8 0.7 0.2"/>
             </geometry>
         </collision>
-        <xacro:inertial_box mass="2" x="0.7" y="0.8" z="0.1">
-            <origin xyz="0.0 0.0 0.0" rpy="0.0 0.0 0.0"/>
-        </xacro:inertial_box>
     </link>
-    <gazebo reference="chassis">
-        <material>Gazebo/Orange</material>
-    </gazebo>
     <joint name="wheel_front_right_joint" type="continuous">
-        <origin xyz="0.20 0.4 0.0" rpy="1.571 0.0 0.0"/>
-        <parent link="chassis"/>
-        <child link="wheel_front_right"/>
+        <origin xyz="0.15 0.4 0.0" rpy="1.57 0.0 0.0"/>
+        <parent link="base_link"/>
+        <child link="wheel_front_right_link"/>
         <axis xyz="0.0 0.0 1.0"/>
     </joint>
-    <link name="wheel_front_right">
-        <visual>
-            <geometry>
-                <cylinder radius="0.15" length="0.1"/>
-            </geometry>
-            <material name="black"/>
-        </visual>
-        <collision>
-            <geometry>
-                <cylinder radius="0.15" length="0.1"/>
-            </geometry>
-        </collision>
-        <xacro:inertial_cylinder mass="2" length="0.1" radius="0.15">
-            <origin xyz="0 0 0" rpy="0 0 0"/>
-        </xacro:inertial_cylinder>
-	</link>
-    <gazebo reference="wheel_front_right">
-        <material>Gazebo/Black</material>
-    </gazebo>
-	<joint name="wheel_front_left_joint" type="continuous">
-        <origin xyz="0.20 -0.4 0.0" rpy="1.571 0.0 0.0"/>
-        <parent link="chassis"/>
-        <child link="wheel_front_left"/>
-        <axis xyz="0.0 0.0 1.0"/>
-    </joint>
-    <link name="wheel_front_left">
+    <link name="wheel_front_right_link">
         <visual>
             <geometry>
@@ -79,18 +54,12 @@
             </geometry>
         </collision>
-        <xacro:inertial_cylinder mass="2" length="0.1" radius="0.15">
-            <origin xyz="0 0 0" rpy="0 0 0"/>
-        </xacro:inertial_cylinder>
     </link>
-    <gazebo reference="wheel_front_left">
-        <material>Gazebo/Black</material>
-    </gazebo>
-    <joint name="wheel_back_right_joint" type="continuous">
-        <origin xyz="-0.20 0.4 0.0" rpy="1.571 0.0 0.0"/>
-        <parent link="chassis"/>
-        <child link="wheel_back_right"/>
+    <joint name="wheel_front_left_joint_joint" type="continuous">
+        <origin xyz="0.15 -0.4 0.0" rpy="1.57 0.0 0.0"/>
+        <parent link="base_link"/>
+        <child link="wheel_front_left_link"/>
         <axis xyz="0.0 0.0 1.0"/>
     </joint>
-    <link name="wheel_back_right">
+    <link name="wheel_front_left_link">
         <visual>
             <geometry>
@@ -101,38 +70,78 @@
         <collision>
             <geometry>
-                <cylinder radius="0.15" length="0.1"/>
+                <cylinder radius="0.15" length="0.15"/>
             </geometry>
         </collision>
-        <xacro:inertial_cylinder mass="2" length="0.1" radius="0.15">
-            <origin xyz="0 0 0" rpy="0 0 0"/>
-        </xacro:inertial_cylinder>
-	</link>
-    <gazebo reference="wheel_back_right">
-        <material>Gazebo/Black</material>
-    </gazebo>
-	<joint name="wheel_back_left_joint" type="continuous">
-        <origin xyz="-0.20 -0.4 0.0" rpy="1.571 0.0 0.0"/>
-        <parent link="chassis"/>
-        <child link="wheel_back_left"/>
-        <axis xyz="0.0 0.0 1.0"/>
+    </link>
+    <joint name="caster_cylinder_joint_joint" type="fixed">
+        <origin xyz="-0.3 0.0 -0.1"/>
+        <parent link="chassis_link"/>
+        <child link="caster_cylinder_link"/>
     </joint>
-    <link name="wheel_back_left">
+    <link name="caster_cylinder_link">
         <visual>
             <geometry>
-                <cylinder radius="0.15" length="0.1"/>
+                <cylinder radius="0.05" length="0.2"/>
             </geometry>
-            <material name="white"/>
+            <material name="black"/>
         </visual>
         <collision>
             <geometry>
-                <cylinder radius="0.15" length="0.1"/>
+                <cylinder radius="0.05" length="0.2"/>
             </geometry>
         </collision>
-        <xacro:inertial_cylinder mass="2" length="0.1" radius="0.15">
-            <origin xyz="0 0 0" rpy="0 0 0"/>
-        </xacro:inertial_cylinder>
     </link>
-    <gazebo reference="wheel_back_left">
-        <material>Gazebo/Black</material>
-    </gazebo>
+    <joint name="caster_joint_joint" type="fixed">
+        <origin xyz="0.0 0.0 -0.1"/>
+        <parent link="caster_cylinder_link"/>
+        <child link="caster_wheel_link"/>
+    </joint>
+    <link name="caster_wheel_link">
+        <visual>
+            <geometry>
+                <sphere  radius="0.05"/>
+            </geometry>
+        </visual>
+        <collision>
+            <geometry>
+                <sphere  radius="0.05"/>
+            </geometry>
+        </collision>
+    </link>
+    <joint name="lidar_joint" type="fixed">
+        <origin xyz="0.0 0.0 0.1"/>
+        <parent link="chassis_link"/>
+        <child link="lidar_link"/>
+    </joint>
+    <link name="lidar_link">
+        <visual>
+            <geometry>
+                <cylinder radius="0.15" length="0.2"/>
+            </geometry>
+            <material name="blue"/>
+        </visual>
+        <collision>
+            <geometry>
+                <cylinder radius="0.15" length="0.2"/>
+            </geometry>
+        </collision>
+    </link>
+    <joint name="camera_joint" type="fixed">
+        <origin xyz="0.41 0.0 0.0"/>
+        <parent link="chassis_link"/>
+        <child link="camera_link"/>
+    </joint>
+    <link name="camera_link">
+        <visual>
+            <geometry>
+                <box size="0.03 0.1 0.1"/>
+            </geometry>
+            <material name="black"/>
+        </visual>
+        <collision>
+            <geometry>
+                <box size="0.05 0.05 0.05"/>
+            </geometry>
+        </collision>
+    </link>
 </robot>

File: ros2_differential_obstacle_robot/src/rover/description/robot.urdf.xacro (robot description, xacro)
@@ -2,7 +2,7 @@
 <robot xmlns:xacro="http://www.ros.org/wiki/xacro" name="rover">
   <xacro:include filename="robot_core.xacro"/>
-  <!-- <xacro:include filename="gazebo_control_skid_steering.xacro"/> -->
+  <xacro:include filename="gazebo_control_skid_steering.xacro"/>
   <xacro:include filename="camera.xacro" />
   <xacro:include filename="lidar.xacro" />
-  <xacro:include filename="gazebo_control_differential_drive.xacro" />
+  <!-- <xacro:include filename="gazebo_control_differential_drive.xacro" /> -->
 </robot>
