Commit message: +update component

File: ros2_differential_drive_robot/install/ros2_differential_drive_robot/share/ros2_differential_drive_robot/urdf/rover.xacro (robot description, xacro)
@@ -30,14 +30,14 @@
             <origin xyz="0.0 0.0 0.0"/>
             <geometry>
+                <box size="0.8 0.7 0.3"/>
+            </geometry>
+            <material name="orange"/>
+        </visual>
+        <collision>
+            <geometry>
                 <box size="0.8 0.7 0.2"/>
             </geometry>
-            <material name="orange"/>
-        </visual>
-        <collision>
-            <geometry>
-                <box size="0.8 0.7 0.2"/>
-            </geometry>
-        </collision>
-        <xacro:inertial_box mass="0.5" x="0.8" y="0.7" z="0.2">
+        </collision>
+        <xacro:inertial_box mass="0.5" x="0.8" y="0.7" z="0.3">
             <origin xyz="0.0 0.0 0.0" rpy="0 0 0"/>
         </xacro:inertial_box>
@@ -150,5 +150,5 @@
     </gazebo>
     <joint name="lidar_joint" type="fixed">
-        <origin xyz="0.0 0.0 0.1"/>
+        <origin xyz="0.0 0.0 0.25" rpy="0 0 0"/>
         <parent link="chassis_link"/>
         <child link="lidar_holder"/>
@@ -158,5 +158,5 @@
         <visual>
             <geometry>
-                <cylinder radius="0.15" length="0.25"/>
+                <cylinder radius="0.05" length="0.25"/>
             </geometry>
             <material name="red"/>
@@ -164,11 +164,14 @@
         <collision>
             <geometry>
-                <cylinder radius="0.15" length="0.25"/>
-            </geometry>
-        </collision>
-        <xacro:inertial_cylinder mass="0.1" length="0.25" radius="0.15">
-            <origin xyz="0 0 0" rpy="0 0 0"/>
-        </xacro:inertial_cylinder>
-    </link>
+                <cylinder radius="0.05" length="0.25"/>
+            </geometry>
+        </collision>
+        <xacro:inertial_cylinder mass="0.1" length="0.25" radius="0.05">
+            <origin xyz="0 0 0" rpy="0 0 0"/>
+        </xacro:inertial_cylinder>
+    </link>
+    <gazebo reference="lidar_holder">
+        <material>Gazebo/Red</material>
+    </gazebo>
      <!-- LIDAR HOLDER -->
      <joint name="lidar_holder_joint" type="fixed">
@@ -181,5 +184,5 @@
         <visual>
             <geometry>
-                <cylinder radius="0.12" length="0.05"/>
+                <cylinder radius="0.1" length="0.05"/>
             </geometry>
             <material name="blue"/>
@@ -187,8 +190,8 @@
         <collision>
             <geometry>
-                <cylinder radius="0.12" length="0.05"/>
-            </geometry>
-        </collision>
-        <xacro:inertial_cylinder mass="0.1" length="0.05" radius="0.12">
+                <cylinder radius="0.1" length="0.05"/>
+            </geometry>
+        </collision>
+        <xacro:inertial_cylinder mass="0.1" length="0.2" radius="0.1">
             <origin xyz="0 0 0" rpy="0 0 0"/>
         </xacro:inertial_cylinder>
@@ -196,5 +199,5 @@
     <!-- CAMERA -->
     <joint name="camera_joint" type="fixed">
-        <origin xyz="0.41 0.0 0.0"/>
+        <origin xyz="0.38 0.0 0.25"/>
         <parent link="chassis_link"/>
         <child link="camera_link"/>
@@ -203,5 +206,5 @@
         <visual>
             <geometry>
-                <box size="0.03 0.1 0.1"/>
+                <box size="0.04 0.1 0.2"/>
             </geometry>
             <material name="black"/>
@@ -209,5 +212,5 @@
         <collision>
             <geometry>
-                <box size="0.05 0.05 0.05"/>
+                <box size="0.05 0.1 0.2"/>
             </geometry>
         </collision>
@@ -219,10 +222,11 @@
           <pose> 0 0 0 0 0 0 </pose>
           <visualize>true</visualize>
-          <update_rate>10.0</update_rate>
+          <update_rate>10</update_rate>
           <ray>
             <scan>
               <horizontal>
                 <samples>360</samples>
-                <resolution>1</resolution>
+                <!-- <resolution>1</resolution> -->
+                <!-- <min_angle>0.00</min_angle> -->
                 <min_angle>0.00</min_angle>
                 <max_angle>3.14</max_angle>
@@ -230,7 +234,9 @@
             </scan>
             <range>
-              <min>0.120</min>
-              <max>3.5</max>
-              <resolution>0.015</resolution>
+              <min>0.3</min>
+              <max>12</max>
+              <!-- <min>0.120</min>
+              <max>3.5</max> -->
+              <!-- <resolution>0.015</resolution> -->
             </range>
           </ray>

File: ros2_differential_drive_robot/src/ros2_differential_drive_robot/description/camera.xacro (robot description, xacro)
@@ -25,5 +25,5 @@
     <material>Gazebo/Red</material>
     <sensor type="camera" name="camera">
-      <!-- <pose>0 0 0 0 0 0</pose> -->
+      <pose>0 0 0 0 0 0</pose>
       <visualize>true</visualize>
       <update_rate>10.0</update_rate>
