Commit message: +added optical link

File: rover/install/rover/share/rover/urdf/rover.xacro (robot description, xacro)
@@ -216,4 +216,10 @@
         </collision>
     </link>
+    <joint name="camera_optical_joint" type="fixed">
+        <parent link="camera_link"/>
+        <child link="camera_link_optical"/>
+        <origin xyz="0 0 0" rpy="${-pi/2} 0 ${-pi/2}"/>
+    </joint>
+    <link name="camera_link_optical"></link>
     <!-- GAZEBO Lidar Plugin -->
     <gazebo reference="lidar_link">

Commit message: +added slam

File: rover/install/rover/share/rover/urdf/rover.xacro (robot description, xacro)
@@ -25,4 +25,11 @@
         <axis xyz="0.0 0.0 0.0"/>
     </joint>
+    <joint name="base_footprint_joint" type="fixed">
+        <origin xyz="0.0 0.0 0.1" rpy="0.0 0.0 0.0"/>
+        <parent link="base_link"/>
+        <child link="base_footprint"/>
+        <axis xyz="0.0 0.0 0.0"/>
+    </joint>
+    <link name="base_footprint"></link>
     <!-- CHASSIS -->
     <link name="chassis_link">

Commit message: +fix my robot urdf

File: rover/install/rover/share/rover/urdf/rover.xacro (robot description, xacro)
@@ -54,5 +54,5 @@
     </gazebo>
     <joint name="wheel_front_right_joint" type="continuous">
-        <origin xyz="0.15 0.4 0.0" rpy="1.57 0.0 0.0"/>
+        <origin xyz="-0.15 0.4 0.0" rpy="1.57 0.0 0.0"/>
         <parent link="base_link"/>
         <child link="wheel_front_right_link"/>
@@ -80,5 +80,5 @@
     </gazebo>
     <joint name="wheel_front_left_joint_joint" type="continuous">
-        <origin xyz="0.15 -0.4 0.0" rpy="1.57 0.0 0.0"/>
+        <origin xyz="-0.15 -0.4 0.0" rpy="1.57 0.0 0.0"/>
         <parent link="base_link"/>
         <child link="wheel_front_left_link"/>
@@ -107,5 +107,5 @@
     <!-- CASTER HOLDER -->
     <joint name="caster_cylinder_joint_joint" type="fixed">
-        <origin xyz="-0.3 0.0 -0.1"/>
+        <origin xyz="0.3 0.0 -0.1"/>
         <parent link="chassis_link"/>
         <child link="caster_cylinder_link"/>
@@ -157,5 +157,5 @@
     </gazebo>
     <joint name="lidar_joint" type="fixed">
-        <origin xyz="0.0 0.0 0.25" rpy="0 0 0"/>
+        <origin xyz="0.0 0.0 0.25" rpy="0 0 1.5708"/>
         <parent link="chassis_link"/>
         <child link="lidar_holder"/>
@@ -183,5 +183,5 @@
      <!-- LIDAR HOLDER -->
      <joint name="lidar_holder_joint" type="fixed">
-        <origin xyz="0.0 0.0 0.15" rpy="0.0 0.0 4.71239"/>
+        <origin xyz="0.0 0.0 0.15" rpy="0.0 0.0 0"/>
         <parent link="lidar_holder"/>
         <child link="lidar_link"/>
@@ -206,5 +206,5 @@
     <!-- CAMERA -->
     <joint name="camera_joint" type="fixed">
-        <origin xyz="0.38 0.0 0.25"/>
+        <origin xyz="-0.38 0.0 0.25" rpy="0 0 ${pi}"/>
         <parent link="chassis_link"/>
         <child link="camera_link"/>
