Commit message: +added ros2_controllers

File: ros2_diff_nav2_slam/install/ros2_diff_nav2_slam/share/ros2_diff_nav2_slam/urdf/diff.robot.xacro (robot description, xacro)
@@ -35,4 +35,5 @@
     </visual>
     <collision>
+        <origin xyz="0.095 0.0 0.0275" rpy="0.0 0.0 0.0"/>
         <geometry>
             <box size="0.19 0.11 0.055"/>
@@ -40,5 +41,5 @@
     </collision>
     <xacro:inertial_box mass="0.1" x="0.19" y="0.11" z="0.055">
-        <origin xyz="0.0 0.0 0.0275" rpy="0 0 0"/>
+        <origin xyz="0.095 0.0 0.0275" rpy="0.0 0.0 0.0"/>
     </xacro:inertial_box>
     </link>
@@ -48,5 +49,5 @@
     <!-- RIGHT WHEEL JOINT -->
     <joint name="right_wheel_joint" type="continuous">
-        <origin xyz="0.0 -0.07 0.0" rpy="-1.57 0.0 0.0"/>
+        <origin xyz="0.0 -0.09 0.0" rpy="-1.57 0.0 0.0"/>
         <parent link="base_link"/>
         <child link="right_wheel_link"/>
@@ -63,5 +64,6 @@
         <collision>
             <geometry>
-                <cylinder radius="0.0325" length="0.025"/>
+                <!-- <cylinder radius="0.0325" length="0.025"/> -->
+                <sphere radius="0.0325"/>
             </geometry>
         </collision>
@@ -75,5 +77,5 @@
     <!-- LEFT WHEEL JOINT -->
     <joint name="left_wheel_joint" type="continuous">
-        <origin xyz="0.0 0.07 0.0" rpy="1.57 0.0 0.0"/>
+        <origin xyz="0.0 0.09 0.0" rpy="1.57 0.0 0.0"/>
         <parent link="base_link"/>
         <child link="left_wheel_link"/>
@@ -90,5 +92,6 @@
         <collision>
             <geometry>
-                <cylinder radius="0.0325" length="0.025"/>
+                <!-- <cylinder radius="0.0325" length="0.025"/> -->
+                <sphere radius="0.0325"/>
             </geometry>
         </collision>

File: ros2_diff_nav2_slam/install/ros2_diff_nav2_slam/share/ros2_diff_nav2_slam/urdf/robot.urdf.xacro (robot description, xacro)
@@ -2,4 +2,5 @@
 <robot xmlns:xacro="http://www.ros.org/wiki/xacro" name="diff_robot">
     <xacro:include filename="diff.robot.xacro"/>
-    <xacro:include filename="gazebo_control_differential_drive.xacro" />
+    <xacro:include filename="ros2_control.xacro" />
+    <!-- <xacro:include filename="gazebo_control_differential_drive.xacro" /> -->
 </robot>
