Commit message: + edit config on wheel and left right

File: techdiffbot/build/techdiffbot/urdf/ros2_control_gazebo.xacro (robot description, xacro)
@@ -1 +1 @@
-/home/jlukas/My_Project/ROS2/techdiffbot/src/techdiffbot/urdf/ros2_control_gazebo.xacro
+/home/jlukas/Desktop/My_Project/ROS2/techdiffbot/src/techdiffbot/urdf/ros2_control_gazebo.xacro

File: techdiffbot/build/techdiffbot/urdf/ros2_control_real_robot.xacro (robot description, xacro)
@@ -1 +1 @@
-/home/jlukas/My_Project/ROS2/techdiffbot/src/techdiffbot/urdf/ros2_control_real_robot.xacro
+/home/jlukas/Desktop/My_Project/ROS2/techdiffbot/src/techdiffbot/urdf/ros2_control_real_robot.xacro

File: techdiffbot/install/techdiffbot/share/techdiffbot/urdf/core.robot.xacro (robot description, xacro)
@@ -47,7 +47,36 @@
         <material>Gazebo/Red</material>
     </gazebo>
+    <!-- LEFT WHEEL JOINT -->
+    <joint name="left_wheel_joint" type="continuous">
+        <origin xyz="0.0 -0.105 0.0" rpy="${pi/2} 0.0 0.0"/>
+        <parent link="base_link"/>
+        <child link="left_wheel_link"/>
+        <axis xyz="0.0 0.0 -1.0"/>
+    </joint>
+    <!-- LEFT WHEEL LINK -->
+    <link name="left_wheel_link">
+        <visual>
+            <geometry>
+                <cylinder radius="0.03405" length="0.027"/>
+                <!-- <cylinder radius="0.03405" length="0.01"/> -->
+            </geometry>
+            <material name="white"/>
+        </visual>
+        <collision>
+            <geometry>
+                <cylinder radius="0.03405" length="0.027"/>
+                <!-- <sphere radius="0.0325"/> -->
+            </geometry>
+        </collision>
+        <xacro:inertial_cylinder mass="0.05" length="0.027" radius="0.03405">
+            <origin xyz="0.0 0.0 -1.0" rpy="${pi/2} 0.0 0.0"/>
+        </xacro:inertial_cylinder>
+    </link>
+    <gazebo reference="left_wheel_link">
+        <material>Gazebo/White</material>
+    </gazebo>
     <!-- RIGHT WHEEL JOINT -->
     <joint name="right_wheel_joint" type="continuous">
-        <origin xyz="0.0 -0.105 0.0" rpy="-1.57 0.0 0.0"/>
+        <origin xyz="0.0 0.105 0.0" rpy="-${pi/2} 0.0 0.0"/>
         <parent link="base_link"/>
         <child link="right_wheel_link"/>
@@ -70,37 +99,8 @@
     </collision>
     <xacro:inertial_cylinder mass="0.05" length="0.027" radius="0.03405">
-        <origin xyz="0.0 0.0 0.0" rpy="0.0 0.0 0.0"/>
+        <origin xyz="0.0 -0.105 0.0" rpy="-${pi/2} 0.0 0.0"/>
     </xacro:inertial_cylinder>
     </link>
     <gazebo reference="right_wheel_link">
-        <material>Gazebo/White</material>
-    </gazebo>
-    <!-- LEFT WHEEL JOINT -->
-    <joint name="left_wheel_joint" type="continuous">
-        <origin xyz="0.0 0.105 0.0" rpy="-1.57 0.0 0.0"/>
-        <parent link="base_link"/>
-        <child link="left_wheel_link"/>
-        <axis xyz="0.0 0.0 1.0"/>
-    </joint>
-    <!-- LEFT WHEEL LINK -->
-    <link name="left_wheel_link">
-        <visual>
-            <geometry>
-                <cylinder radius="0.03405" length="0.027"/>
-                <!-- <cylinder radius="0.03405" length="0.01"/> -->
-            </geometry>
-            <material name="white"/>
-        </visual>
-        <collision>
-            <geometry>
-                <cylinder radius="0.03405" length="0.027"/>
-                <!-- <sphere radius="0.0325"/> -->
-            </geometry>
-        </collision>
-        <xacro:inertial_cylinder mass="0.05" length="0.027" radius="0.03405">
-            <origin xyz="0.0 0.0 0.0" rpy="0.0 0.0 0.0"/>
-        </xacro:inertial_cylinder>
-    </link>
-    <gazebo reference="left_wheel_link">
         <material>Gazebo/White</material>
     </gazebo>
