Commit message: +added line gazebo.sim.launc.py to automatically open the saved world

File: techdiffbot/build/techdiffbot/urdf/core.robot.xacro (robot description, xacro)
@@ -1 +1 @@
-/home/jlukas/ROS2/techdiffbot/src/techdiffbot/urdf/core.robot.xacro
+/home/jlukas/Desktop/My_Project/ROS2/techdiffbot/src/techdiffbot/urdf/core.robot.xacro

File: techdiffbot/build/techdiffbot/urdf/diff.robot.urdf.xacro (robot description, xacro)
@@ -1 +1 @@
-/home/jlukas/ROS2/techdiffbot/src/techdiffbot/urdf/diff.robot.urdf.xacro
+/home/jlukas/Desktop/My_Project/ROS2/techdiffbot/src/techdiffbot/urdf/diff.robot.urdf.xacro

File: techdiffbot/build/techdiffbot/urdf/gazebo_control.xacro (robot description, xacro)
@@ -1 +1 @@
-/home/jlukas/ROS2/techdiffbot/src/techdiffbot/urdf/gazebo_control.xacro
+/home/jlukas/Desktop/My_Project/ROS2/techdiffbot/src/techdiffbot/urdf/gazebo_control.xacro

File: techdiffbot/build/techdiffbot/urdf/inertial_macros.xacro (robot description, xacro)
@@ -1 +1 @@
-/home/jlukas/ROS2/techdiffbot/src/techdiffbot/urdf/inertial_macros.xacro
+/home/jlukas/Desktop/My_Project/ROS2/techdiffbot/src/techdiffbot/urdf/inertial_macros.xacro

File: techdiffbot/build/techdiffbot/urdf/real.robot.gazebo.sim.xacro (robot description, xacro)
@@ -1 +1 @@
-/home/jlukas/ROS2/techdiffbot/src/techdiffbot/urdf/real.robot.gazebo.sim.xacro
+/home/jlukas/Desktop/My_Project/ROS2/techdiffbot/src/techdiffbot/urdf/real.robot.gazebo.sim.xacro

File: techdiffbot/build/techdiffbot/urdf/ros2_control.xacro (robot description, xacro)
@@ -1 +1 @@
-/home/jlukas/ROS2/techdiffbot/src/techdiffbot/urdf/ros2_control.xacro
+/home/jlukas/Desktop/My_Project/ROS2/techdiffbot/src/techdiffbot/urdf/ros2_control.xacro

File: techdiffbot/build/techdiffbot/urdf/ros2_control_gazebo.xacro (robot description, xacro)
@@ -1 +1 @@
-/home/jlukas/ROS2/techdiffbot/src/techdiffbot/urdf/ros2_control_gazebo.xacro
+/home/jlukas/Desktop/My_Project/ROS2/techdiffbot/src/techdiffbot/urdf/ros2_control_gazebo.xacro

File: techdiffbot/install/diffdrive_arduino/share/diffdrive_arduino/ros2_control/diffbot.ros2_control.xacro (robot description, xacro)
@@ -1 +1 @@
-/home/jlukas/ROS2/techdiffbot/src/diffdrive_arduino/description/ros2_control/diffbot.ros2_control.xacro
+/home/jlukas/Desktop/My_Project/ROS2/techdiffbot/src/diffdrive_arduino/description/ros2_control/diffbot.ros2_control.xacro

File: techdiffbot/install/diffdrive_arduino/share/diffdrive_arduino/urdf/diffbot.materials.xacro (robot description, xacro)
@@ -1 +1 @@
-/home/jlukas/ROS2/techdiffbot/src/diffdrive_arduino/description/urdf/diffbot.materials.xacro
+/home/jlukas/Desktop/My_Project/ROS2/techdiffbot/src/diffdrive_arduino/description/urdf/diffbot.materials.xacro

File: techdiffbot/install/diffdrive_arduino/share/diffdrive_arduino/urdf/diffbot.urdf.xacro (robot description, xacro)
@@ -1 +1 @@
-/home/jlukas/ROS2/techdiffbot/src/diffdrive_arduino/description/urdf/diffbot.urdf.xacro
+/home/jlukas/Desktop/My_Project/ROS2/techdiffbot/src/diffdrive_arduino/description/urdf/diffbot.urdf.xacro

File: techdiffbot/install/diffdrive_arduino/share/diffdrive_arduino/urdf/diffbot_description.urdf.xacro (robot description, xacro)
@@ -1 +1 @@
-/home/jlukas/ROS2/techdiffbot/src/diffdrive_arduino/description/urdf/diffbot_description.urdf.xacro
+/home/jlukas/Desktop/My_Project/ROS2/techdiffbot/src/diffdrive_arduino/description/urdf/diffbot_description.urdf.xacro

File: techdiffbot/install/techdiffbot/share/techdiffbot/urdf/core.robot.xacro (robot description, xacro)
@@ -19,4 +19,12 @@
     <!-- BASE LINK -->
     <link name="base_link"></link>
+    <!-- BASE FOOTPRINT LINK -->
+    <link name="base_footprint"></link>
+    <!-- BASE FOOTPRINT JOINT -->
+    <joint name="base_footprint_joint" type="fixed">
+        <parent link="base_link"/>
+        <child link="base_footprint"/>
+        <origin xyz="0 0 0" rpy="0 0 0"/>
+    </joint>
     <!-- CHASSIS JOINT -->
     <joint name="chassis_joint" type="fixed">
