Commit message: added serial and diffdrive package

File: techdiffbot/src/techdiffbot/urdf/ros2_control_real_robot.xacro (robot description, xacro)
@@ -13,5 +13,5 @@
         </hardware>
         <!-- Note everything below here is the same as the Gazebo one -->
-        <joint name="left_wheel_joint">
+        <joint name="right_wheel_joint">
             <command_interface name="velocity">
                 <param name="min">-10</param>
@@ -21,5 +21,5 @@
             <state_interface name="velocity"/>
         </joint>
-        <joint name="right_wheel_joint">
+        <joint name="left_wheel_joint">
             <command_interface name="velocity">
                 <param name="min">-10</param>
