Commit message: -modify the yaml file with correct wheel assignment

File: techdiffbot/install/techdiffbot/share/techdiffbot/urdf/core.robot.xacro (robot description, xacro)
@@ -49,5 +49,5 @@
     <!-- LEFT WHEEL JOINT -->
     <joint name="left_wheel_joint" type="continuous">
-        <origin xyz="0.0 -0.105 0.0" rpy="${pi/2} 0.0 0.0"/>
+        <origin xyz="0.0 0.105 0.0" rpy="${pi/2} 0.0 0.0"/>
         <parent link="base_link"/>
         <child link="left_wheel_link"/>
@@ -78,5 +78,5 @@
     <!-- RIGHT WHEEL JOINT -->
     <joint name="right_wheel_joint" type="continuous">
-        <origin xyz="0.0 0.105 0.0" rpy="-${pi/2} 0.0 0.0"/>
+        <origin xyz="0.0 -0.105 0.0" rpy="-${pi/2} 0.0 0.0"/>
         <parent link="base_link"/>
         <child link="right_wheel_link"/>

Commit message: +modify motor whell

File: techdiffbot/install/techdiffbot/share/techdiffbot/urdf/core.robot.xacro (robot description, xacro)
@@ -49,5 +49,5 @@
     <!-- LEFT WHEEL JOINT -->
     <joint name="left_wheel_joint" type="continuous">
-        <origin xyz="0.0 0.105 0.0" rpy="${pi/2} 0.0 0.0"/>
+        <origin xyz="0.0 0.105 0.0" rpy="-${pi/2} 0.0 0.0"/>
         <parent link="base_link"/>
         <child link="left_wheel_link"/>
@@ -70,5 +70,5 @@
         </collision>
         <xacro:inertial_cylinder mass="0.05" length="0.027" radius="0.03405">
-            <origin xyz="0.0 0.0 -1.0" rpy="${pi/2} 0.0 0.0"/>
+            <origin xyz="0.0 0.0 0.0" rpy="0.0 0.0 0.0"/>
         </xacro:inertial_cylinder>
     </link>
@@ -78,5 +78,5 @@
     <!-- RIGHT WHEEL JOINT -->
     <joint name="right_wheel_joint" type="continuous">
-        <origin xyz="0.0 -0.105 0.0" rpy="-${pi/2} 0.0 0.0"/>
+        <origin xyz="0.0 -0.105 0.0" rpy="${pi/2} 0.0 0.0"/>
         <parent link="base_link"/>
         <child link="right_wheel_link"/>
@@ -99,5 +99,5 @@
     </collision>
     <xacro:inertial_cylinder mass="0.05" length="0.027" radius="0.03405">
-        <origin xyz="0.0 -0.105 0.0" rpy="-${pi/2} 0.0 0.0"/>
+        <origin xyz="0.0 0.0 0.0" rpy="0.0 0.0 0.0"/>
     </xacro:inertial_cylinder>
     </link>

Commit message: -remove sign

File: techdiffbot/install/techdiffbot/share/techdiffbot/urdf/core.robot.xacro (robot description, xacro)
@@ -52,5 +52,5 @@
         <parent link="base_link"/>
         <child link="left_wheel_link"/>
-        <axis xyz="0.0 0.0 -1.0"/>
+        <axis xyz="0.0 0.0 1.0"/>
     </joint>
     <!-- LEFT WHEEL LINK -->
@@ -81,5 +81,5 @@
         <parent link="base_link"/>
         <child link="right_wheel_link"/>
-        <axis xyz="0.0 0.0 1.0"/>
+        <axis xyz="0.0 0.0 -1.0"/>
     </joint>
     <!-- RIGHT WHEEL LINK -->

Commit message: this version work with physical roboto

File: techdiffbot/install/techdiffbot/share/techdiffbot/urdf/core.robot.xacro (robot description, xacro)
@@ -150,8 +150,9 @@
         <origin xyz="0.0 0.0 0.1" rpy="0.0 0.0 0.0"/>
         <parent link="chassis_link"/>
-        <child link="lidar_case_link"/>
+	<!-- <child link="lidar_case_link"/> -->
+        <child link="ldlidar_base"/>
     </joint>
     <!-- LIDAR CASE LINK -->
-    <link name="lidar_case_link">
+    <link name="ldlidar_base">
     <visual>
         <!-- <origin xyz="0.0 0.0 0.0" rpy="0.0 0.0 0.0"/> -->
@@ -170,5 +171,11 @@
     </xacro:inertial_box>
     </link>
-    <gazebo reference="lidar_case_link">
+     <joint name="ldlidar_link_joint" type="fixed">
+        <parent link="ldlidar_base"/>
+        <child link="ldlidar_link"/>
+        <origin xyz="0.0 0.0 0.0" rpy="0.0 0.0 0.0" />
+    </joint>
+    <link name="ldlidar_link"/>
+    <gazebo reference="ldlidar_base">
         <material>Gazebo/Red</material>
     </gazebo>
@@ -176,5 +183,5 @@
     <joint name="lidar_joint" type="fixed">
         <origin xyz="0.0 0.0 0.055 " rpy="0.0 0.0 4.71239"/>
-        <parent link="lidar_case_link"/>
+        <parent link="ldlidar_base"/>
         <child link="lidar_link"/>
     </joint>

File: techdiffbot/install/techdiffbot/share/techdiffbot/urdf/ros2_control.xacro (robot description, xacro)
@@ -8,5 +8,5 @@
                 <param name="right_wheel_name">right_wheel_joint</param>
                 <param name="loop_rate">30</param>
-                <param name="device">/dev/ttyUSB0</param>
+                <param name="device">/dev/serial/by-path/platform-fd500000.pcie-pci-0000:01:00.0-usb-0:1.2:1.0-port0</param>
                 <param name="baud_rate">57600</param>
                 <param name="timeout_ms">1000</param>

Commit message: added working simulation robot

File: techdiffbot/install/techdiffbot/share/techdiffbot/urdf/core.robot.xacro (robot description, xacro)
@@ -147,14 +147,12 @@
     <link name="camera_link_optical"></link>
     <!-- LIDAR CASE JOINT -->
-    <joint name="lidar_case_joint" type="fixed">
+    <joint name="lidar_joint" type="fixed">
+        <parent link="chassis_link"/>
+        <child link="ldlidar_base"/>
         <origin xyz="0.0 0.0 0.1" rpy="0.0 0.0 0.0"/>
-        <parent link="chassis_link"/>
-	<!-- <child link="lidar_case_link"/> -->
-        <child link="ldlidar_base"/>
     </joint>
     <!-- LIDAR CASE LINK -->
     <link name="ldlidar_base">
     <visual>
-        <!-- <origin xyz="0.0 0.0 0.0" rpy="0.0 0.0 0.0"/> -->
         <geometry>
             <box size="0.08 0.18 0.095"/>
@@ -171,15 +169,9 @@
     </xacro:inertial_box>
     </link>
-     <joint name="ldlidar_link_joint" type="fixed">
-        <parent link="ldlidar_base"/>
-        <child link="ldlidar_link"/>
-        <origin xyz="0.0 0.0 0.0" rpy="0.0 0.0 0.0" />
-    </joint>
-    <link name="ldlidar_link"/>
     <gazebo reference="ldlidar_base">
         <material>Gazebo/Red</material>
     </gazebo>
     <!-- LIDAR  JOINT -->
-    <joint name="lidar_joint" type="fixed">
+    <joint name="lidar_case_joint" type="fixed">
         <origin xyz="0.0 0.0 0.055 " rpy="0.0 0.0 4.71239"/>
         <parent link="ldlidar_base"/>

Commit message: added physical robot configuration

File: techdiffbot/install/techdiffbot/share/techdiffbot/urdf/core.robot.xacro (robot description, xacro)
@@ -176,8 +176,8 @@
         <origin xyz="0.0 0.0 0.055 " rpy="0.0 0.0 4.71239"/>
         <parent link="ldlidar_base"/>
-        <child link="lidar_link"/>
+        <child link="ldlidar_link"/>
     </joint>
     <!-- LIDAR LINK -->
-    <link name="lidar_link">
+    <link name="ldlidar_link">
     <visual>
         <!-- <origin xyz="0.0 0.0 0.0" rpy="0.0 0.0 0.0"/> -->
@@ -196,5 +196,5 @@
     </xacro:inertial_cylinder>
     </link>
-    <gazebo reference="lidar_link">
+    <gazebo reference="ldlidar_link">
         <material>Gazebo/Blue</material>
     </gazebo>
@@ -256,5 +256,5 @@
     </gazebo>
     <!-- GAZEBO Lidar Plugin -->
-    <gazebo reference="lidar_link">
+    <gazebo reference="ldlidar_link">
         <material>Gazebo/Blue</material>
         <sensor name="laser" type="ray">
@@ -290,5 +290,5 @@
             </ros>
             <output_type>sensor_msgs/LaserScan</output_type>
-            <frame_name>lidar_link</frame_name>
+            <frame_name>ldlidar_link</frame_name>
             </plugin>
         </sensor>
