Commit message: added lidar slamtech command

File: techdiffbot/install/diffdrive_arduino/share/diffdrive_arduino/ros2_control/diffbot.ros2_control.xacro (robot description, xacro)
@@ -1,31 +1 @@
-<?xml version="1.0"?>
-<robot xmlns:xacro="http://www.ros.org/wiki/xacro">
-  <xacro:macro name="diffbot_ros2_control" params="name prefix">
-    <ros2_control name="${name}" type="system">
-      <hardware>
-        <plugin>diffdrive_arduino/DiffDriveArduinoHardware</plugin>
-        <param name="left_wheel_name">left_wheel_joint</param>
-        <param name="right_wheel_name">right_wheel_joint</param>
-        <param name="loop_rate">30</param>
-        <param name="device">/dev/serial/by-path/platform-fd500000.pcie-pci-0000:01:00.0-usb-0:1.3:1.0-port0</param>
-        <param name="baud_rate">57600</param>
-        <param name="timeout_ms">1000</param>
-        <param name="enc_counts_per_rev">3436</param>
-        <param name="pid_p">20</param>
-        <param name="pid_d">12</param>
-        <param name="pid_i">0</param>
-        <param name="pid_o">50</param>
-      </hardware>
-      <joint name="${prefix}left_wheel_joint">
-        <command_interface name="velocity"/>
-        <state_interface name="position"/>
-        <state_interface name="velocity"/>
-      </joint>
-      <joint name="${prefix}right_wheel_joint">
-        <command_interface name="velocity"/>
-        <state_interface name="position"/>
-        <state_interface name="velocity"/>
-      </joint>
-    </ros2_control>
-  </xacro:macro>
-</robot>
+/home/ros2/Desktop/My_Project/ROS2/techdiffbot/src/diffdrive_arduino/description/ros2_control/diffbot.ros2_control.xacro

File: techdiffbot/install/diffdrive_arduino/share/diffdrive_arduino/urdf/diffbot.materials.xacro (robot description, xacro)
@@ -1,31 +1 @@
-<?xml version="1.0"?>
-<!--
-Copied from ROS1 example:
-https://github.com/ros-simulation/gazebo_ros_demos/blob/kinetic-devel/rrbot_description/urdf/materials.xacro
--->
-<robot>
-  <material name="black">
-    <color rgba="0.0 0.0 0.0 1.0"/>
-  </material>
-  <material name="blue">
-    <color rgba="0.0 0.0 0.8 1.0"/>
-  </material>
-  <material name="green">
-    <color rgba="0.0 0.8 0.0 1.0"/>
-  </material>
-  <material name="grey">
-    <color rgba="0.2 0.2 0.2 1.0"/>
-  </material>
-  <material name="orange">
-    <color rgba="${255/255} ${108/255} ${10/255} 1.0"/>
-  </material>
-  <material name="brown">
-    <color rgba="${222/255} ${207/255} ${195/255} 1.0"/>
-  </material>
-  <material name="red">
-    <color rgba="0.8 0.0 0.0 1.0"/>
-  </material>
-  <material name="white">
-    <color rgba="1.0 1.0 1.0 1.0"/>
-  </material>
-</robot>
+/home/ros2/Desktop/My_Project/ROS2/techdiffbot/src/diffdrive_arduino/description/urdf/diffbot.materials.xacro

File: techdiffbot/install/diffdrive_arduino/share/diffdrive_arduino/urdf/diffbot.urdf.xacro (robot description, xacro)
@@ -1,13 +1 @@
-<?xml version="1.0"?>
-<!-- Basic differential drive mobile base -->
-<robot xmlns:xacro="http://www.ros.org/wiki/xacro" name="diffdrive_robot">
-  <xacro:arg name="prefix" default="" />
-  <xacro:include filename="$(find diffdrive_arduino)/urdf/diffbot_description.urdf.xacro" />
-  <!-- Import Rviz colors -->
-  <xacro:include filename="$(find diffdrive_arduino)/urdf/diffbot.materials.xacro" />
-  <!-- Import diffbot ros2_control description -->
-  <xacro:include filename="$(find diffdrive_arduino)/ros2_control/diffbot.ros2_control.xacro" />
-  <xacro:diffbot prefix="$(arg prefix)" />
-  <xacro:diffbot_ros2_control
-    name="DiffBot" prefix="$(arg prefix)" />
-</robot>
+/home/ros2/Desktop/My_Project/ROS2/techdiffbot/src/diffdrive_arduino/description/urdf/diffbot.urdf.xacro

File: techdiffbot/install/diffdrive_arduino/share/diffdrive_arduino/urdf/diffbot_description.urdf.xacro (robot description, xacro)
@@ -1,161 +1 @@
-<?xml version="1.0"?>
-<robot xmlns:xacro="http://www.ros.org/wiki/xacro">
-  <xacro:macro name="diffbot" params="prefix">
-  <!-- Constants for robot dimensions -->
-  <xacro:property name="PI" value="3.1415926535897931"/>
-  <xacro:property name="base_mass" value="0.3" /> <!-- arbitrary value for base mass -->
-  <xacro:property name="base_width" value="0.1" />
-  <xacro:property name="base_length" value="0.1" />
-  <xacro:property name="base_height" value="0.05" />
-  <xacro:property name="wheel_mass" value="0.3" /> <!-- arbitrary value for wheel mass -->
-  <xacro:property name="wheel_len" value="0.020" />
-  <xacro:property name="wheel_radius" value="0.015" />
-  <xacro:property name="caster_wheel_mass" value="0.1" /> <!-- arbitrary value for caster wheel mass -->
-  <xacro:property name="caster_wheel_radius" value="0.015" />
-  <xacro:property name="z_offset" value="-${base_height/2}" /> <!-- Space btw top of beam and the each joint -->
-  <!-- Base Link -->
-  <link name="${prefix}base_link">
-    <collision>
-      <origin xyz="0 0 0" rpy="0 0 0"/>
-      <geometry>
-        <box size="${base_width} ${base_length} ${base_height}"/>
-      </geometry>
-    </collision>
-    <visual>
-      <origin xyz="0 0 ${base_height/2}" rpy="0 0 0"/>
-      <geometry>
-        <box size="${base_width} ${base_length} ${base_height}"/>
-      </geometry>
-      <material name="orange"/>
-    </visual>
-    <inertial>
-      <origin xyz="0 0 0" rpy="0 0 0"/>
-      <mass value="${base_mass}"/>
-      <inertia
-        ixx="${base_mass / 12.0 * (base_length*base_length + base_height*base_height)}" ixy="0.0" ixz="0.0"
-        iyy="${base_mass / 12.0 * (base_height*base_height + base_width*base_width)}" iyz="0.0"
-        izz="${base_mass / 12.0 * (base_width*base_width + base_length*base_length)}"/>
-      </inertial>
-    </link>
-    <joint name="${prefix}left_wheel_joint" type="continuous">
-      <parent link="${prefix}base_link"/>
-      <child link="${prefix}left_wheel"/>
-      <origin xyz="0 -${base_width/2} ${z_offset}" rpy="0 0 0"/>
-      <axis xyz="0 1 0"/>
-      <dynamics damping="0.2"/>
-    </joint>
-    <!-- left wheel Link -->
-    <link name="${prefix}left_wheel">
-      <collision>
-        <origin xyz="0 0 0" rpy="${PI/2} 0 0"/>
-        <geometry>
-          <cylinder length="${wheel_len}" radius="${wheel_radius}"/>
-        </geometry>
-      </collision>
-      <visual>
-        <origin xyz="0 0 0" rpy="${PI/2} 0 0"/>
-        <geometry>
-          <cylinder length="${wheel_len}" radius="${wheel_radius}"/>
-        </geometry>
-        <material name="black"/>
-      </visual>
-      <inertial>
-        <origin xyz="0 0 0" rpy="${PI/2} 0 0"/>
-        <mass value="${wheel_mass}"/>
-        <inertia
-          ixx="${wheel_mass / 12.0 * (3*wheel_radius + wheel_len*wheel_len)}" ixy="0.0" ixz="0.0"
-          iyy="${wheel_mass / 12.0 * wheel_radius*wheel_radius}" iyz="0.0"
-          izz="${wheel_mass / 12.0 * wheel_radius*wheel_radius}"/>
-        </inertial>
-      </link>
-    <joint name="${prefix}right_wheel_joint" type="continuous">
-      <parent link="${prefix}base_link"/>
-      <child link="${prefix}right_wheel"/>
-      <origin xyz="0 ${base_width/2} ${z_offset}" rpy="0 0 0"/>
-      <axis xyz="0 1 0"/>
-      <dynamics damping="0.2"/>
-    </joint>
-    <!-- right wheel Link -->
-    <link name="${prefix}right_wheel">
-      <collision>
-        <origin xyz="0 0 0" rpy="${PI/2} 0 0"/>
-        <geometry>
-          <cylinder length="${wheel_len}" radius="${wheel_radius}"/>
-        </geometry>
-      </collision>
-      <visual>
-        <origin xyz="0 0 0" rpy="${PI/2} 0 0"/>
-        <geometry>
-          <cylinder length="${wheel_len}" radius="${wheel_radius}"/>
-        </geometry>
-        <material name="black"/>
-      </visual>
-      <inertial>
-        <origin xyz="0 0 0" rpy="${PI/2} 0 0"/>
-        <mass value="${wheel_mass}"/>
-        <inertia
-          ixx="${wheel_mass / 12.0 * (3*wheel_radius + wheel_len*wheel_len)}" ixy="0.0" ixz="0.0"
-          iyy="${wheel_mass / 12.0 * wheel_radius*wheel_radius}" iyz="0.0"
-          izz="${wheel_mass / 12.0 * wheel_radius*wheel_radius}"/>
-        </inertial>
-      </link>
-    <joint name="${prefix}caster_frontal_wheel_joint" type="fixed">
-      <parent link="${prefix}base_link"/>
-      <child link="${prefix}caster_frontal_wheel"/>
-      <origin xyz="${base_width/2 - caster_wheel_radius} 0 ${z_offset}" rpy="0 0 0"/>
-    </joint>
-    <!-- caster frontal wheel Link -->
-    <link name="${prefix}caster_frontal_wheel">
-      <collision>
-        <origin xyz="0 0 0" rpy="0 0 0"/>
-        <geometry>
-          <sphere radius="${caster_wheel_radius}"/>
-        </geometry>
-      </collision>
-      <visual>
-        <origin xyz="0 0 0" rpy="0 0 0"/>
-        <geometry>
-          <sphere radius="${caster_wheel_radius}"/>
-        </geometry>
-        <material name="white"/>
-      </visual>
-      <inertial>
-        <origin xyz="0 0 0" rpy="0 0 0"/>
-        <mass value="${caster_wheel_mass}"/>
-        <inertia
-          ixx="${caster_wheel_mass * 0.4 * (caster_wheel_radius * caster_wheel_radius)}" ixy="0.0" ixz="0.0"
-          iyy="${caster_wheel_mass * 0.4 * (caster_wheel_radius * caster_wheel_radius)}" iyz="0.0"
-          izz="${caster_wheel_mass * 0.4 * (caster_wheel_radius * caster_wheel_radius)}"/>
-        </inertial>
-      </link>
-    <joint name="${prefix}caster_rear_wheel_joint" type="fixed">
-      <parent link="${prefix}base_link"/>
-      <child link="${prefix}caster_rear_wheel"/>
-      <origin xyz="${-base_width/2 + caster_wheel_radius} 0 ${z_offset}" rpy="0 0 0"/>
-    </joint>
-    <!-- caster rear wheel Link -->
-    <link name="${prefix}caster_rear_wheel">
-      <collision>
-        <origin xyz="0 0 0" rpy="0 0 0"/>
-        <geometry>
-          <sphere radius="${caster_wheel_radius}"/>
-        </geometry>
-      </collision>
-      <visual>
-        <origin xyz="0 0 0" rpy="0 0 0"/>
-        <geometry>
-          <sphere radius="${caster_wheel_radius}"/>
-        </geometry>
-        <material name="white"/>
-      </visual>
-      <inertial>
-        <origin xyz="0 0 0" rpy="0 0 0"/>
-        <mass value="${caster_wheel_mass}"/>
-        <inertia
-          ixx="${caster_wheel_mass * 0.4 * (caster_wheel_radius * caster_wheel_radius)}" ixy="0.0" ixz="0.0"
-          iyy="${caster_wheel_mass * 0.4 * (caster_wheel_radius * caster_wheel_radius)}" iyz="0.0"
-          izz="${caster_wheel_mass * 0.4 * (caster_wheel_radius * caster_wheel_radius)}"/>
-        </inertial>
-      </link>
-  </xacro:macro>
-</robot>
+/home/ros2/Desktop/My_Project/ROS2/techdiffbot/src/diffdrive_arduino/description/urdf/diffbot_description.urdf.xacro

File: techdiffbot/install/techdiffbot/share/techdiffbot/urdf/core.robot.xacro (robot description, xacro)
@@ -1,333 +1 @@
-<?xml version="1.0"?>
-<robot xmlns:xacro="http://www.ros.org/wiki/xacro" name="diff_robot">
-    <xacro:include filename="inertial_macros.xacro"/>
-    <material name="white">
-        <color rgba="1 1 1 1"/>
-    </material>
-    <material name="orange">
-        <color rgba="1 0.3 0.1 1"/>
-    </material>
-    <material name="blue">
-        <color rgba="0.2 0.2 1 1"/>
-    </material>
-    <material name="black">
-        <color rgba="0 0 0 1"/>
-    </material>
-    <material name="red">
-        <color rgba="1 0 0 1"/>
-    </material>
-    <!-- BASE LINK -->
-    <link name="base_link"></link>
-    <!-- BASE FOOTPRINT JOINT -->
-    <joint name="base_footprint_joint" type="fixed">
-        <parent link="base_link"/>
-        <child link="base_footprint"/>
-        <origin xyz="0 0 0" rpy="0 0 0"/>
-    </joint>
-     <!-- BASE FOOTPRINT LINK -->
-     <link name="base_footprint"></link>
-    <!-- CHASSIS JOINT -->
-    <joint name="chassis_joint" type="fixed">
-        <parent link="base_link"/>
-        <child link="chassis_link"/>
-        <origin xyz="-0.04 0 0"/> <!-- 18/2 = 9 and -5 = 4cm because of dc motor distance and convert to cm to m = 0.04 -->
-    </joint>
-    <!-- CHASSIS LINK -->
-    <link name="chassis_link">
-    <visual>
-        <origin xyz="0.0 0.0 0.0325" rpy="0.0 0.0 0.0"/>
-        <geometry>
-            <box size="0.18 0.18 0.065"/>
-        </geometry>
-        <material name="red"/>
-    </visual>
-    <collision>
-        <origin xyz="0.0 0.0 0.0325" rpy="0.0 0.0 0.0"/>
-        <geometry>
-            <box size="0.18 0.18 0.065"/>
-        </geometry>
-    </collision>
-    <xacro:inertial_box mass="0.5" x="0.18" y="0.18" z="0.065">
-        <origin xyz="0.0 0.0 0.0325" rpy="0.0 0.0 0.0"/>
-    </xacro:inertial_box>
-    </link>
-    <gazebo reference="chassis_link">
-        <material>Gazebo/Red</material>
-    </gazebo>
-    <!-- LEFT WHEEL JOINT -->
-    <joint name="left_wheel_joint" type="continuous">
-        <origin xyz="0.0 0.105 0.0" rpy="-${pi/2} 0.0 0.0"/>
-        <parent link="base_link"/>
-        <child link="left_wheel_link"/>
-        <axis xyz="0.0 0.0 1.0"/>
-    </joint>
-    <!-- LEFT WHEEL LINK -->
-    <link name="left_wheel_link">
-        <visual>
-            <geometry>
-                <cylinder radius="0.03405" length="0.027"/>
-                <!-- <cylinder radius="0.03405" length="0.01"/> -->
-            </geometry>
-            <material name="white"/>
-        </visual>
-        <collision>
-            <geometry>
-                <cylinder radius="0.03405" length="0.027"/>
-                <!-- <sphere radius="0.0325"/> -->
-            </geometry>
-        </collision>
-        <xacro:inertial_cylinder mass="0.05" length="0.027" radius="0.03405">
-            <origin xyz="0.0 0.0 0.0" rpy="0.0 0.0 0.0"/>
-        </xacro:inertial_cylinder>
-    </link>
-    <gazebo reference="left_wheel_link">
-        <material>Gazebo/White</material>
-    </gazebo>
-    <!-- RIGHT WHEEL JOINT -->
-    <joint name="right_wheel_joint" type="continuous">
-        <origin xyz="0.0 -0.105 0.0" rpy="${pi/2} 0.0 0.0"/>
-        <parent link="base_link"/>
-        <child link="right_wheel_link"/>
-        <axis xyz="0.0 0.0 -1.0"/>
-    </joint>
-    <!-- RIGHT WHEEL LINK -->
-    <link name="right_wheel_link">
-    <visual>
-        <geometry>
-            <cylinder radius="0.03405" length="0.027"/>
-            <!-- <cylinder radius="0.03405" length="0.01"/> -->
-        </geometry>
-        <material name="white"/>
-    </visual>
-    <collision>
-        <geometry>
-            <cylinder radius="0.03405" length="0.027"/>
-            <!-- <sphere radius="0.0325"/> -->
-        </geometry>
-    </collision>
-    <xacro:inertial_cylinder mass="0.05" length="0.027" radius="0.03405">
-        <origin xyz="0.0 0.0 0.0" rpy="0.0 0.0 0.0"/>
-    </xacro:inertial_cylinder>
-    </link>
-    <gazebo reference="right_wheel_link">
-        <material>Gazebo/White</material>
-    </gazebo>
-    <!-- CAMERA JOINT -->
-    <joint name="camera_joint" type="fixed">
-        <origin xyz="0.065 0.0 0.105" rpy="0.0 0.0 0.0"/>
-        <parent link="chassis_link"/>
-        <child link="camera_link"/>
-    </joint>
-    <!-- CAMERA LINK -->
-    <link name="camera_link">
-        <visual>
-            <origin xyz="0.0 0.0 0.0" rpy="0.0 0.0 0.0"/>
-            <geometry>
-                <box size="0.014 0.04 0.08"/>
-            </geometry>
-            <material name="blue"/>
-        </visual>
-        <collision>
-            <geometry>
-                <box size="0.014 0.04 0.08"/>
-            </geometry>
-        </collision>
-        <xacro:inertial_box mass="0.01" x="0.014" y="0.04" z="0.08">
-            <origin xyz="0.0 0.0 0.0" rpy="0.0 0.0 0.0"/>
-        </xacro:inertial_box>
-    </link>
-    <gazebo reference="camera_link">
-        <material>Gazebo/Blue</material>
-    </gazebo>
-    <joint name="camera_optical_joint" type="fixed">
-        <parent link="camera_link"/>
-        <child link="camera_link_optical"/>
-        <origin xyz="0 0 0" rpy="${-pi/2} 0 ${-pi/2}"/>
-    </joint>
-    <link name="camera_link_optical"></link>
-    <!-- LIDAR CASE JOINT -->
-    <joint name="lidar_joint" type="fixed">
-        <parent link="chassis_link"/>
-        <child link="ldlidar_base"/>
-        <origin xyz="0.0 0.0 0.1" rpy="0.0 0.0 0.0"/>
-    </joint>
-    <!-- LIDAR CASE LINK -->
-    <link name="ldlidar_base">
-    <visual>
-        <geometry>
-            <box size="0.08 0.18 0.095"/>
-        </geometry>
-        <material name="red"/>
-    </visual>
-    <collision>
-        <geometry>
-            <box size="0.08 0.18 0.095"/>
-        </geometry>
-    </collision>
-    <xacro:inertial_box mass="0.03" x="0.08" y="0.18" z="0.095">
-        <origin xyz="0.0 0.0 0.0" rpy="0.0 0.0 0.0"/>
-    </xacro:inertial_box>
-    </link>
-    <gazebo reference="ldlidar_base">
-        <material>Gazebo/Red</material>
-    </gazebo>
-    <!-- LIDAR  JOINT -->
-    <joint name="lidar_case_joint" type="fixed">
-        <origin xyz="0.0 0.0 0.055 " rpy="0.0 0.0 4.71239"/>
-        <parent link="ldlidar_base"/>
-        <child link="ldlidar_link"/>
-    </joint>
-    <!-- LIDAR LINK -->
-    <link name="ldlidar_link">
-    <visual>
-        <!-- <origin xyz="0.0 0.0 0.0" rpy="0.0 0.0 0.0"/> -->
-        <geometry>
-            <cylinder radius="0.0175" length="0.0175"/>
-        </geometry>
-        <material name="blue"/>
-    </visual>
-    <collision>
-        <geometry>
-            <cylinder radius="0.0175" length="0.0175"/>
-        </geometry>
-    </collision>
-    <xacro:inertial_cylinder mass="0.1" length="0.0175" radius="0.0175">
-        <origin xyz="0.0 0.0 0.0" rpy="0.0 0.0 0.0"/>
-    </xacro:inertial_cylinder>
-    </link>
-    <gazebo reference="ldlidar_link">
-        <material>Gazebo/Blue</material>
-    </gazebo>
-    <!-- CASTER HOLDER JOINT -->
-    <joint name="caster_holder_joint" type="fixed">
-        <origin xyz="-0.06 0.0 0.0" rpy="0.0 0.0 0.0"/>
-        <parent link="chassis_link"/>
-        <child link="caster_holder_link"/>
-    </joint>
-    <!-- CASTER HOLDER LINK -->
-    <link name="caster_holder_link">
-        <visual>
-            <origin xyz="0.0 0.0 0.0" rpy="0.0 0.0 0.0"/>
-            <geometry>
-                <cylinder radius="0.0175" length="0.040"/>
-            </geometry>
-            <material name="white"/>
-        </visual>
-        <collision>
-            <geometry>
-                <cylinder radius="0.0175" length="0.040"/>
-            </geometry>
-        </collision>
-        <xacro:inertial_cylinder mass="0.01" length="0.040" radius="0.0175">
-        <origin xyz="0.0 0.0 0.0" rpy="0.0 0.0 0.0"/>
-        </xacro:inertial_cylinder>
-    </link>
-    <gazebo reference="caster_holder_link">
-        <material>Gazebo/White</material>
-    </gazebo>
-    <!-- CASTER BALL JOINT -->
-    <joint name="caster_ball_joint" type="fixed">
-        <origin xyz="0.0 0.0 -0.020" rpy="0.0 0.0 0.0"/>
-        <parent link="caster_holder_link"/>
-        <child link="caster_link"/>
-    </joint>
-    <!-- CASTER BALL LINK -->
-    <link name="caster_link">
-    <visual>
-        <origin xyz="0.0 0.0 0.0" rpy="0.0 0.0 0.0"/>
-        <geometry>
-            <sphere radius="0.0125"/>
-        </geometry>
-        <material name="white"/>
-    </visual>
-    <collision>
-        <geometry>
-            <sphere radius="0.0125"/>
-        </geometry>
-    </collision>
-    <xacro:inertial_sphere mass="0.01" radius="0.0125">
-        <origin xyz="0.0 0.0 0.0" rpy="0.0 0.0 0.0"/>
-    </xacro:inertial_sphere>
-    </link>
-    <gazebo reference="caster_link">
-        <material>Gazebo/White</material>
-        <mu1 value="0.001"/>
-        <mu2 value="0.001"/>
-    </gazebo>
-    <!-- GAZEBO Lidar Plugin -->
-    <gazebo reference="ldlidar_link">
-        <material>Gazebo/Blue</material>
-        <sensor name="laser" type="ray">
-            <pose> 0 0 0 0 0 0 </pose>
-            <visualize>true</visualize>
-            <update_rate>10</update_rate>
-            <ray>
-                <scan>
-                    <horizontal>
-                    <samples>360</samples>
-                    <!-- <resolution>1</resolution> -->
-                    <!-- <min_angle>0.00</min_angle> -->
-                    <min_angle>-3.14</min_angle>
-                    <max_angle>3.14</max_angle>
-                    <!-- <min_angle>0.00</min_angle>
-                    <max_angle>3.14</max_angle>  -->
-                    <!-- <max_angle>6.28319</max_angle>  -->
-                    <!-- 3.14 is 180 degree -->
-                  </horizontal>
-                </scan>
-                <range>
-                    <min>0.3</min>
-                    <max>12</max>
-                    <!-- <min>0.120</min>
-                    <max>3.5</max> -->
-                    <!-- <resolution>0.015</resolution> -->
-                </range>
-            </ray>
-            <plugin name="laser_controller" filename="libgazebo_ros_ray_sensor.so">
-            <ros>
-                <remapping>~/out:=scan</remapping>
-                <!-- <argument>~/out:=scan</argument> -->
-            </ros>
-            <output_type>sensor_msgs/LaserScan</output_type>
-            <frame_name>ldlidar_link</frame_name>
-            </plugin>
-        </sensor>
-    </gazebo>
-    <!-- CAMERA  Plugin -->
-    <gazebo reference="camera_link">
-        <material>Gazebo/Black</material>
-        <sensor type="camera" name="camera">
-        <pose>0 0 0 0 0 0</pose>
-        <visualize>true</visualize>
-        <update_rate>10.0</update_rate>
-        <camera name="head">
-            <horizontal_fov>1.089</horizontal_fov>
-            <image>
-                <width>640</width>
-                <height>480</height>
-                <format>R8G8B8</format>
-            </image>
-            <clip>
-                <near>0.05</near>
-                <far>8.0</far>
-            </clip>
-        </camera>
-        <!-- <plugin name="camera_controller" filename="libgazebo_ros_camera.so">
-            <alwaysOn>true</alwaysOn>
-            <updateRate>0.0</updateRate>
-            <imageTopicName>image_raw</imageTopicName>
-            <cameraInfoTopicName>camera_info</cameraInfoTopicName>
-            <frameName>camera_link_optical</frameName>
-            <hackBaseline>0.07</hackBaseline>
-            <distortionK1>0.0</distortionK1>
-            <distortionK2>0.0</distortionK2>
-            <distortionK3>0.0</distortionK3>
-            <distortionT1>0.0</distortionT1>
-            <distortionT2>0.0</distortionT2>
-        </plugin> -->
-        <plugin name="camera_controller" filename="libgazebo_ros_camera.so">
-            <frame_name>camera_link_optical</frame_name>
-        </plugin>
-        </sensor>
-    </gazebo>
-</robot>
+/home/ros2/Desktop/My_Project/ROS2/techdiffbot/build/techdiffbot/urdf/core.robot.xacro
